File: KiCad_Data/Complex Op Amps - Project 2 - Part 2.kicad_pcb (KiCad board)
At the start: 2 copper layers, 184.2 x 81.5 mm, 95 parts, among them P1 Potentiometer P/N: 3590P-2-**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, P2 Potentiometer P/N: 3590P-2-**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, SW1 SPST Switch, P/N: GT12MABE, SW2 SPST Switch, P/N: GT12MABE, SW3 SPST Switch, P/N: GT12MABE, SW4 SPST Switch, P/N: GT12MABE, SW5 SPST Switch, P/N: GT12MABE, T1 Transistor P/N: 2N3906, T2 Transistor P/N: 2N3906, T3 Transistor P/N: 2N3906, T4 Transistor P/N: 2N3906

Commit message: Made small corrections regarding ground fill
Parts:
- moved R14 1.27 mm to (136.5, 101.6)
- moved OPAMP8 1.27 mm to (125.7, 124.5)
- moved R38 0.59 mm to (132.2, 105.4)
- moved OPAMP9 0.50 mm to (134.6, 113.0)
- moved R12 0.20 mm to (121.9, 92.5)
Routing:
- net Net-(R31-Pad2): track 0.00 -> 57.4 mm, vias 0 -> 1
- net +5V: track 190.9 -> 237.4 mm
- net -15V: track 521.5 -> 548.0 mm
- net +15V: track 774.5 -> 765.7 mm
- net Net-(R14-Pad1): track 14.4 -> 16.3 mm
- net Net-(OPAMP8--): track 207.7 -> 209.1 mm
- net Net-(R18-Pad1): track 199.1 -> 197.9 mm
- net Net-(T3-B): track 71.6 -> 72.5 mm
- net Net-(TR2-B): track 221.8 -> 222.5 mm
- net Net-(T1-B): track 191.1 -> 191.8 mm
- net Net-(OPAMP5-+): track 54.5 -> 54.0 mm
- net Net-(OPAMP9--): track 4.15 -> 3.65 mm
Other:
- board text added: "Samarpreet Bhatti & Dr. Martin June 15 2023 Generic Circuit"
