File: KiCad_Data/Complex Op Amps - Project 2 - Part 2.kicad_sch (KiCad schematic)
At the start: 128 parts, among them P1 50k, P2 50k, SW1 SPDT Switch, P/N: 7101SD9AV2BE, SW2 SPDT Switch, P/N: 7101SD9AV2BE, SW3 SPDT Switch, P/N: 7101SD9AV2BE, SW4 SPDT Switch, P/N: 7101SD9AV2BE, SW5 SPDT Switch, P/N: 7101SD9AV2BE, SW6 SPDT Switch, P/N: 7101SD9AV2BE, SW7 SPDT Switch, P/N: 7101SD9AV2BE, T1 Transistor P/N: 2N3906, T2 Transistor P/N: 2N3906, T3 Transistor P/N: 2N3906, T4 Transistor P/N: 2N3906

Commit message: Updated IDC connections
Connections:
- net GND: now also IDC1.7 (C); no longer IDC1.5 (C)
- net at OPAMP6.6, R15.2: now also IDC1.6 (C); no longer IDC1.7 (C)
- net at OPAMP11.6, R35.2: now also IDC1.5 (C); no longer IDC1.6 (C)
Changed lines of the file:
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@@
     (stroke (width 0) (type default))
   )
+  (wire (pts (xy 34.925 138.43) (xy 42.545 138.43))
+    (stroke (width 0) (type default))
+  )
   (wire (pts (xy 239.395 147.955) (xy 239.395 165.1))
     (stroke (width 0) (type default))
@@
     (stroke (width 0) (type default))
   )
-  (wire (pts (xy 44.45 142.24) (xy 34.925 142.24))
+  (wire (pts (xy 32.385 137.795) (xy 44.45 137.795))
     (stroke (width 0) (type default))
   )
@@
     (stroke (width 0) (type default))
   )
-  (wire (pts (xy 34.925 142.24) (xy 34.925 145.415))
-    (stroke (width 0) (type default))
-  )
   (wire (pts (xy 229.235 58.42) (xy 235.585 58.42))
     (stroke (width 0) (type default))
@@
     (stroke (width 0) (type default))
   )
+  (wire (pts (xy 32.385 137.795) (xy 32.385 145.415))
+    (stroke (width 0) (type default))
+  )
   (wire (pts (xy 83.82 154.94) (xy 84.455 154.94))
     (stroke (width 0) (type default))
@@
     (stroke (width 0) (type default))
   )
-  (wire (pts (xy 44.45 173.99) (xy 44.45 142.24))
+  (wire (pts (xy 44.45 173.99) (xy 44.45 137.795))
     (stroke (width 0) (type default))
   )
@@
     (stroke (width 0) (type default))
   )
+  (wire (pts (xy 34.925 145.415) (xy 34.925 138.43))
+    (stroke (width 0) (type default))
+  )
   (wire (pts (xy 70.485 142.24) (xy 77.47 142.24))
     (stroke (width 0) (type default))
@@
     (stroke (width 0) (type default))
   )
-  (wire (pts (xy 42.545 179.07) (xy 42.545 145.415))
+  (wire (pts (xy 42.545 138.43) (xy 42.545 179.07))
     (stroke (width 0) (type default))
   )
@@
     (stroke (width 0) (type default))
   )
-  (wire (pts (xy 42.545 145.415) (xy 37.465 145.415))
-    (stroke (width 0) (type default))
-  )
   (wire (pts (xy 243.205 34.29) (xy 243.205 39.37))
     (stroke (width 0) (type default))
@@
     (effects (font (size 1.27 1.27)) (justify left bottom))
   )
-  (text "Current Out" (at 34.29 142.24 0)
+  (text "Current Out" (at 34.29 137.795 0)
     (effects (font (size 1.27 1.27)) (justify left bottom))
   )
@@
     )
   )
+  (symbol (lib_id "power:GND") (at 37.465 145.415 180) (unit 1)
+    (in_bom yes) (on_board yes) (dnp no)
+    (property "Reference" "#PWR063" (at 37.465 139.065 0)
+      (effects (font (size 1.27 1.27)) hide)
+    )
+    (property "Value" "GND" (at 37.465 142.24 0)
+      (effects (font (size 1.27 1.27)))
+    )
+    (property "Footprint" "" (at 37.465 145.415 0)
+      (effects (font (size 1.27 1.27)) hide)
+    )
+    (property "Datasheet" "" (at 37.465 145.415 0)
+      (effects (font (size 1.27 1.27)) hide)
+    )
+    (pin "1")
+    (instances
+      (project "Complex Op Amps - Project 2 - Part 2"
+        (path "/630740a9-e2c4-4754-9b7b-0b1cb79935b3"
+          (reference "#PWR063") (unit 1)
+        )
+      )
+    )
+  )
   (symbol (lib_id "Complex_Op_Amps_Footprints:Resistor") (at 222.885 87.63 90) (unit 1)
     (in_bom yes) (on_board yes) (dnp no) (fields_autoplaced)
@@
         )
       )
-    )
-  )
-  (symbol (lib_id "power:GND") (at 32.385 145.415 180) (unit 1)
-    (in_bom yes) (on_board yes) (dnp no)
-    (property "Reference" "#PWR063" (at 32.385 139.065 0)
-      (effects (font (size 1.27 1.27)) hide)
-    )
-    (property "Value" "GND" (at 32.385 141.605 0)
-      (effects (font (size 1.27 1.27)))
-    )
-    (property "Footprint" "" (at 32.385 145.415 0)
-      (effects (font (size 1.27 1.27)) hide)
-    )
-    (property "Datasheet" "" (at 32.385 145.415 0)
-      (effects (font (size 1.27 1.27)) hide)
-    )
-    (pin "1")
-    (instances
-      (project "Complex Op Amps - Project 2 - Part 2"
-        (path "/630740a9-e2c4-4754-9b7b-0b1cb79935b3"
-          (reference "#PWR063") (unit 1)
-        )
-      )
